Commit message: changed ruedas

File: src/mi_robot_mecanum/urdf/mi_robot.urdf.xacro (robot description, xacro)
@@ -60,5 +60,5 @@
       </collision>
       <inertial>
-      <origin xyz="0 0 0.02" rpy="0 0 0"/>
+      <origin xyz="0 0 0.02" rpy="${pi/2} 0 0"/>
       <mass value="${rueda_masa}"/>
       <xacro:inercia_cilindro m="${rueda_masa}" r="${rueda_radio}" h="${rueda_ancho}"/>
@@ -68,5 +68,5 @@
       <parent link="base_link"/>
       <child link="rueda_${prefijo}"/>
-      <origin xyz="x_signo*lx, y_signo*ly, 0" rpy="-3.14/2 0 0"/>
+      <origin xyz="${x_signo*lx}, ${y_signo*ly}, 0" rpy="${pi/2} 0 0"/>
     </joint>
   </xacro:macro>

Commit message: fixed positions and cleaned pi values

File: src/mi_robot_mecanum/urdf/mi_robot.urdf.xacro (robot description, xacro)
@@ -60,13 +60,14 @@
       </collision>
       <inertial>
-      <origin xyz="0 0 0.02" rpy="${pi/2} 0 0"/>
+      <origin xyz="0 0 0" rpy="0 0 0"/>
       <mass value="${rueda_masa}"/>
       <xacro:inercia_cilindro m="${rueda_masa}" r="${rueda_radio}" h="${rueda_ancho}"/>
     </inertial>
     </link>
-    <joint name="joint_rueda${prefijo}" type="continous">
+    <joint name="joint_rueda_${prefijo}" type="continuous">
       <parent link="base_link"/>
       <child link="rueda_${prefijo}"/>
-      <origin xyz="${x_signo*lx}, ${y_signo*ly}, 0" rpy="${pi/2} 0 0"/>
+      <origin xyz="${x_signo*lx} ${y_signo*ly} 0" rpy="${-pi/2} 0 0"/>
+      <axis xyz="0 0 1"/>
     </joint>
   </xacro:macro>
@@ -78,14 +79,14 @@
   <link name="lidar_link">
       <visual>
-        <origin xyz="0.06 0 0.13" rpy="0 0 0"/>
+        <origin xyz="0 0 0" rpy="0 0 0"/>
         <geometry><cylinder radius="${0.076}" length="${0.041}"/></geometry>
         <material name="negro"><color rgba="0.1 0.1 0.1 1"/></material>
       </visual>
       <collision>
-        <origin xyz="0.06 0 0.13" rpy="0 0 0"/>
+        <origin xyz="0 0 0" rpy="0 0 0"/>
         <geometry><cylinder radius="${0.076}" length="${0.041}"/></geometry>
       </collision>
       <inertial>
-      <origin xyz="0 0 0.02" rpy="0 0 0"/>
+      <origin xyz="0 0 0" rpy="0 0 0"/>
       <mass value="${0.19}"/>
       <xacro:inercia_cilindro m="${0.19}" r="${0.076}" h="${0.041}"/>
@@ -124,14 +125,14 @@
 <link name="camara_link">
     <visual>
-      <origin xyz="0.16 0 0.09" rpy="0 0 0"/>
+      <origin xyz="0 0 0" rpy="0 0 0"/>
       <geometry><box size="${0.04} ${0.165} ${0.048}"/></geometry>
       <material name="negro"><color rgba="0.1 0.1 0.1 1"/></material>
     </visual>
     <collision>
-      <origin xxyz="0.16 0 0.09" rpy="0 0 0"/>
+      <origin xyz="0 0 0" rpy="0 0 0"/>
       <geometry><box size="${0.04} ${0.165} ${0.048}"/></geometry>
     </collision>
     <inertial>
-      <origin xyz="0.16 0 0.09" rpy="0 0 0"/>
+      <origin xyz="0 0 0" rpy="0 0 0"/>
       <mass value="${0.31}"/>
       <xacro:inercia_caja m="${0.31}" x="${0.04}" y="${0.165}" z="${0.048}"/>
@@ -141,33 +142,16 @@
     <parent link="base_link"/>
     <child link="camara_link"/>
-    <origin xyz="0.10 0 0.20" rpy="0 0 0"/>
+    <origin xyz="0.16 0 0.09" rpy="0 0 0"/>
   </joint>
-  <link name="camara_optica_link">
-    <visual>
-      <origin xyz="0.16 0 0.09" rpy="-3.14/2 0 -3.14/2"/>
-      <geometry><box size="${0.04} ${0.165} ${0.048}"/></geometry>
-      <material name="negro"><color rgba="0.1 0.1 0.1 1"/></material>
-    </visual>
-    <collision>
-      <origin xxyz="0.16 0 0.09" rpy="-3.14/2 0 -3.14/2"/>
-      <geometry><box size="${0.04} ${0.165} ${0.048}"/></geometry>
-    </collision>
-    <inertial>
-      <origin xyz="0.16 0 0.09" rpy="-3.14/2 0 -3.14/2"/>
-      <mass value="${0.31}"/>
-      <xacro:inercia_caja m="${0.31}" x="${0.04}" y="${0.165}" z="${0.048}"/>
-    </inertial>
-  </link>
+  <link name="camara_optica_link"/>
   <joint name="joint_camara_optica" type="fixed">
     <parent link="camara_link"/>
     <child link="camara_optica_link"/>
-    <origin xyz="0.10 0 0.20" rpy="-3.14/2 0 -3.14/2"/>
+    <origin xyz="0 0 0" rpy="${-pi/2} 0 ${-pi/2}"/>
   </joint>
-  <!-- TODO: link "camara_optica_link" y joint fijo "joint_camara_optica" desde
-       camara_link con rpy = (-π/2, 0, -π/2) (REP-103) -->
   <gazebo reference="camara_link">
     <sensor name="astra" type="rgbd_camera">
       <topic>/camara</topic>
-      <gz_frame_id>camera_link</gz_frame_id>
+      <gz_frame_id>camara_optica_link</gz_frame_id>
       <update_rate>30</update_rate>
       <always_on>1</always_on>
